File: projects/odrive/kicad/odrive-v3.5/odrive-v3.5.kicad_sch (KiCad schematic)
At the start: 0 parts

Commit message: Build the ODrive v3.5 and v4 schematics, both verified
The v3.5 recreation (Top + MotorCell M0/M1 + AuxHalfH) matches the netlist
ground truth extracted from the Altium PDF's embedded text layer — every
component, value and net membership diffed clean, ERC 0 errors. The v4
schematic implements docs/v4-design.md across 10 block sheets, 375 parts,
ERC 0 errors, with the STM32 pin map verified pin-by-pin against v3.5;
only the design doc's declared changes differ (PA2/PA3 SO3 jumpers,
PB2/PB10 mux selects, PC4 mux common).

Both were built through Konnect MCP tools by the e2e workflow's oracle
loops; the v4 ERC count converged 740 -> 579 -> 144 -> 2 -> 0 across five
fix rounds. The project sym-lib-tables pin absolute /nix/store paths and
need re-registering if the kicad pin moves; the schematics embed their
symbols, so they open regardless. Details in docs/LOG.md; layout and fab
outputs are the remaining phases.
Parts:
- added C1: 270pF, symbol Device:C
- added C10, C22, C6, C62, C7, C8, C9: 100nF, symbol Device:C
- added C11, C12, C13, C14, C15, C16, C17, C18: 470uF, symbol Device:C_Polarized
- added C19, C20, C21, C26, C40, C44, C55, C68: 4.7uF, symbol Device:C
- added C2, C3: 10pF, symbol Device:C
- added C4, C5, C65: 2.2uF, symbol Device:C
- added C63, C64, C66, C67, C69: 82pF, symbol Device:C
- added FID1, FID2, FID3, FID4: (no value), symbol Mechanical:Fiducial
- added H1, H10, H11, H12, H2, H3, H4, H5, H6, H7, H8, H9: (no value), symbol Mechanical:MountingHole
- added J1: (no value), symbol /home/aldo/Dev/aldoborrero/cad/.claude/worktrees/odrive/projects/odrive/kicad/o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
- added J10, J15, J20, J24, J25, J26, J27, J28, J5, J6: (no value), symbol Jumper:SolderJumper_2_Open
- added J2: Header 6, symbol Connector_Generic:Conn_01x06
- added J3: Leftheader, symbol Connector_Generic:Conn_01x20
- added J4: Rightheader, symbol Connector_Generic:Conn_01x12
- added J7, J8: (no value), symbol Connector_Generic:Conn_01x01
- added J9: (no value), symbol Connector_Generic:Conn_01x02
- added LED1: Green, symbol /home/aldo/Dev/aldoborrero/cad/.claude/worktrees/odrive/projects/odrive/kicad/o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
- added NT1: Net Tie, symbol Device:NetTie_2
- added R1, R2, R3, R4: 22R, symbol Device:R
- added R10, R11, R32, R33, R34, R52, R53, R55, R56, R57, R59, R60, R9: 3.3k, symbol Device:R
- added R5: 120R, symbol Device:R
- added R58, R7: 1k, symbol Device:R
- added R6: 10K, symbol Device:R
- added R8: 47K, symbol Device:R
- added SW1: (no value), symbol Switch:SW_DIP_x02
- added TP1, TP2, TP3, TP4, TP5: (no value), symbol Connector:TestPoint
- added U1: SN65HVD232DR, symbol /home/aldo/Dev/aldoborrero/cad/.claude/worktrees/odrive/projects/odrive/kicad/o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
- added U2: STM32F405RGT6, symbol MCU_ST_STM32F4:STM32F405RGTx
- added U3, U8: 3.3V, symbol /home/aldo/Dev/aldoborrero/cad/.claude/worktrees/odrive/projects/odrive/kicad/o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
- added XT1: 8 MHz, symbol /home/aldo/Dev/aldoborrero/cad/.claude/worktrees/odrive/projects/odrive/kicad/o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
Connections:
- new net 5V: C65.2, J2.1 (Pin_1), J4.2 (Pin_2), J4.8 (Pin_8), U3.3 (VIN), U8.1 (VIN), U8.3 (ON/OFF)
- new net AGND: C1.1, C21.1, C22.2, J3.7 (Pin_7), NT1.2, R7.1, TP5.1, U2.12 (VSSA), U8.2 (GND)
- new net AUX_H: R59.1, U2.30 (PB11)
- new net AUX_L: R60.1, U2.29 (PB10)
- new net AUX_TEMP: U2.21 (PA5)
- new net AVCC: C21.2, C22.1, J3.6 (Pin_6), TP4.1, U2.13 (VDDA), U8.4 (NC), U8.5 (VOUT)
- new net BOOT0: R8.1, SW1.3, U2.60 (BOOT0)
- new net CAN_D: U1.1 (D), U2.62 (PB9)
- new net CAN_H: J3.3 (Pin_3), R5.1, U1.7 (CANH)
- new net CAN_L: J3.4 (Pin_4), SW1.1, U1.6 (CANL)
- new net CAN_R: U1.4 (R), U2.61 (PB8)
- new net DCBUS: C11.1, C12.1, C13.1, C14.1, C15.1, C16.1, C17.1, C18.1, C26.2, C40.2, C44.2, C55.2, C68.2, J7.1 (Pin_1), J9.2 (Pin_2), R6.2
- new net EN_GATE: U2.33 (PB12)
- new net GND: C10.2, C19.1, C2.2, C20.1, C3.2, C4.1, C5.1, C6.1, C62.2, C63.2, C64.2, C65.1, C66.2, C67.2, C69.2, C7.2, C8.2, C9.2, J1.5 (GND), J1.SH (Shield), J2.4 (Pin_4), J3.19 (Pin_19), J3.2 (Pin_2), J3.20 (Pin_20), J3.5 (Pin_5), J4.12 (Pin_12), J4.6 (Pin_6), NT1.1, R58.2, R59.2, R60.2, SW1.2, TP3.1, U1.2 (GND), U2.18 (VSS), U2.63 (VSS), U3.1 (GND), XT1.G (GND)
- new net GPIO_1: J3.11 (Pin_11), J5.1 (A), R52.2
- new net GPIO_1_FLT: J5.2 (B), J6.2 (B), R52.1, U2.14 (PA0)
- new net GPIO_2: J10.1 (A), J3.12 (Pin_12), R53.2
- new net GPIO_2_FLT: J10.2 (B), J15.2 (B), R53.1, U2.15 (PA1)
- new net GPIO_3: J3.13 (Pin_13), U2.16 (PA2)
- new net GPIO_4: J3.14 (Pin_14), U2.17 (PA3)
- new net GPIO_5: J3.15 (Pin_15), U2.24 (PC4)
- new net GPIO_6: J27.1 (A), J3.16 (Pin_16), R57.2
- new net GPIO_6_FLT: J27.2 (B), J28.2 (B), R57.1, U2.28 (PB2)
- new net GPIO_7: J20.1 (A), J3.17 (Pin_17), R55.2
- new net GPIO_7_FLT: J20.2 (B), J24.2 (B), R55.1, U2.50 (PA15)
- new net GPIO_8: J25.1 (A), J3.18 (Pin_18), R56.2
- new net GPIO_8_FLT: J25.2 (B), J26.2 (B), R56.1, U2.55 (PB3)
- new net M0_AH: U2.41 (PA8)
- new net M0_AL: U2.34 (PB13)
- new net M0_BH: U2.42 (PA9)
- new net M0_BL: U2.35 (PB14)
- new net M0_CH: U2.43 (PA10)
- new net M0_CL: U2.36 (PB15)
- new net M0_ENC_A: J4.9 (Pin_9), R9.1, U2.56 (PB4)
- new net M0_ENC_B: J4.10 (Pin_10), R10.1, U2.57 (PB5)
- new net M0_ENC_Z: J4.11 (Pin_11), R11.1, U2.40 (PC9)
- new net M0_SO1: U2.8 (PC0)
- new net M0_SO2: U2.9 (PC1)
- new net M0_TEMP: U2.25 (PC5)
- new net M0_nCS: U2.2 (PC13)
- new net M1_AH: U2.37 (PC6)
- new net M1_AL: U2.23 (PA7)
- new net M1_BH: U2.38 (PC7)
- new net M1_BL: U2.26 (PB0)
- new net M1_CH: U2.39 (PC8)
- new net M1_CL: U2.27 (PB1)
- new net M1_ENC_A: J4.3 (Pin_3), R32.2, U2.58 (PB6)
- new net M1_ENC_B: J4.4 (Pin_4), R33.2, U2.59 (PB7)
- new net M1_ENC_Z: J4.5 (Pin_5), R34.2, U2.4 (PC15)
- new net M1_SO1: U2.11 (PC3)
- new net M1_SO2: U2.10 (PC2)
- new net M1_TEMP: U2.20 (PA4)
- new net M1_nCS: U2.3 (PC14)
- new net NetC2_1: C2.1, U2.6 (PH1), XT1.1 (X1)
- new net NetC3_1: C3.1, U2.5 (PH0), XT1.3 (X2)
- new net NetC4_2: C4.2, U2.47 (VCAP_2)
- new net NetC5_2: C5.2, U2.31 (VCAP_1)
- new net NetC63_1: C63.1, J6.1 (A)
- new net NetC64_1: C64.1, J15.1 (A)
- new net NetC66_1: C66.1, J24.1 (A)
- new net NetC67_1: C67.1, J26.1 (A)
- new net NetC69_1: C69.1, J28.1 (A)
- new net NetJ1_2: J1.2 (D-), R1.2, TP1.1
- new net NetJ1_3: J1.3 (D+), R3.2, TP2.1
- new net NetJ2_3: J2.3 (Pin_3), R2.1
- new net NetJ2_5: J2.5 (Pin_5), R4.1
- new net NetLED1_K: LED1.K, R58.1
- new net NetR5_2: R5.2, SW1.4
- new net PGND: C11.2, C12.2, C13.2, C14.2, C15.2, C16.2, C17.2, C18.2, C26.1, C40.1, C44.1, C55.1, C68.1, J8.1 (Pin_1), J9.1 (Pin_1)
- new net SPI_MISO: J3.9 (Pin_9), U2.52 (PC11)
- new net SPI_MOSI: J3.10 (Pin_10), U2.53 (PC12)
- new net SPI_SCK: J3.8 (Pin_8), U2.51 (PC10)
- new net SWCLK: R2.2, U2.49 (PA14)
- new net SWDIO: R4.2, U2.46 (PA13)
- new net USB_DM: R1.1, U2.44 (PA11)
- new net USB_DP: R3.1, U2.45 (PA12)
- new net VBUS_S: C1.2, R6.1, R7.2, U2.22 (PA6)
- new net VCC: C10.1, C19.2, C20.2, C62.1, C7.1, C8.1, C9.1, J2.2 (Pin_2), J3.1 (Pin_1), J4.1 (Pin_1), J4.7 (Pin_7), LED1.A, R10.2, R11.2, R32.1, R33.1, R34.1, R8.2, R9.2, U1.3 (VCC), U2.1 (VBAT), U2.19 (VDD), U2.32 (VDD), U2.48 (VDD), U2.64 (VDD), U3.2 (VOUT), U3.4 (VOUT_TAB)
- new net nFAULT: U2.54 (PD2)
- new net nRST: C6.2, J2.6 (Pin_6), U2.7 (NRST)
- no-connect marks 0 -> 7
Other:
- added sheet Aux (AuxHalfH.kicad_sch)
- added sheet Motor 0 (MotorCell.kicad_sch)
- added sheet Motor 1 (MotorCell_noPow.kicad_sch)
