File: projects/odrive/kicad/odrive-v4/can.kicad_sch (KiCad schematic)
At the start: 17 parts, among them J7 JST-GH-4 CAN, J8 JST-GH-4 CAN, SW1 CAN_TERM, U32 TPS2553DBV, U34 TCAN1042HGV

Commit message: Make the v4 schematic sheets readable, netlist-invariant
The verified v4 schematic was electrically perfect and visually unreadable:
connectivity lived in labels stuck on pins, text overlapped, and parts sat
on the title block. Reworked all ten block sheets through Konnect: real
wires for local connections, labels kept for power rails and inter-sheet
nets, parts grouped by function, junction dots where wires join.

The invariant was enforced, not assumed: the exported netlist is diffed
against a reference frozen before the rework - 378 components and 283 nets,
identical membership pin by pin - and ERC holds at 0 errors. The lesson
that forced the rework is now a standing gate: numeric oracles (ERC,
netlist diff, overlap counts) all passed on the unreadable version, so
every sheet is also rendered to PNG and looked at before being declared
done.

An interrupted fix round left one known cosmetic issue, documented in
docs/LOG.md: the encoders-gpio GPIO group's reference/value text fields
float ~134mm right of their symbols, over the title block. konnect 0.2.2
has no tool that repositions property fields, so it waits for 0.11.0.
Also adds the fab footprints the sheets reference (MEGA fuse, Phoenix
terminal blocks, CMC) and restores the board file to the blank template -
the aborted layout skeleton was not worth keeping.
Parts:
- C132, C133, C134, C135: footprint (none) -> Capacitor_SMD:C_0603_1608Metric
- C136: footprint (none) -> Capacitor_SMD:C_0805_2012Metric
- D22: footprint (none) -> Package_TO_SOT_SMD:SOT-23
- FB3: footprint (none) -> odrive_footprints:L_CommonMode_Murata_DLW32SH101XF2
- J7, J8: footprint (none) -> Connector_JST:JST_GH_BM04B-GHS-TBT_1x04-1MP_P1.25mm_Vertical
- R127, R128, R129, R130, R131: footprint (none) -> Resistor_SMD:R_0603_1608Metric
- SW1: footprint (none) -> Button_Switch_THT:SW_DIP_SPSTx01_Slide_9.78x4.72mm_W7.62mm_P2.54mm
- U32: footprint (none) -> Package_TO_SOT_SMD:SOT-23-6
- U34: footprint (none) -> Package_SO:SOIC-8_3.9x4.9mm_P1.27mm
Other:
- note added: "5V AUX POWER SWITCH"
- note added: "CAN CONNECTORS"
- note added: "CAN TRANSCEIVER"
- note added: "SPLIT TERMINATION"
Changed lines of the file:
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@@
+    (diameter 0)
+)
+  (junction
+    (at 81.28 35.56)
+    (diameter 0)
+)
+  (junction
+    (at 86.36 35.56)
+    (diameter 0)
+)
+  (junction
+    (at 134.62 35.56)
+    (diameter 0)
+)
+  (junction
+    (at 93.98 86.36)
+    (diameter 0)
+)
+  (junction
+    (at 91.44 91.44)
+    (diameter 0)
+)
+  (junction
+    (at 113.03 86.36)
+    (diameter 0)
+)
+  (junction
+    (at 114.3 91.44)
+    (diameter 0)
+)
+  (junction
+    (at 127 113.03)
     (diameter 0)
 )
@@
       (justify right bottom))
 )
-  (label "CAN_TSPLIT"
-    (at 132.08 113.03 0)
+  (label "CAN_TERM_SW"
+    (at 127 125.73 0)
     (effects
       (font
@@
       (justify left bottom))
 )
-  (label "CAN_TERM_SW"
-    (at 127 125.73 0)
+  (label "CANH"
+    (at 165.1 100.33 90)
     (effects
       (font
@@
       (justify left bottom))
 )
-  (label "CANH"
-    (at 165.1 100.33 90)
+  (label "CANL"
+    (at 170.18 100.33 90)
     (effects
       (font
@@
       (justify left bottom))
 )
-  (label "CANL"
-    (at 170.18 100.33 90)
-    (effects
-      (font
-        (size 1.27 1.27))
-      (justify left bottom))
-)
   (label "CANH"
     (at 185.42 78.74 180)
@@
   (label "CANL"
     (at 185.42 101.6 180)
+    (effects
+      (font
+        (size 1.27 1.27))
+      (justify right bottom))
+)
+  (label "CAN_TSPLIT"
+    (at 127 113.03 180)
     (effects
       (font
@@
         (font
           (size 1.27 1.27))))
-    (property "Footprint" ""
+    (property "Footprint" "Package_SO:SOIC-8_3.9x4.9mm_P1.27mm"
       (at 78.74 88.9 0)
       (hide yes)
@@
         (font
           (size 1.27 1.27))))
-    (property "Footprint" ""
+    (property "Footprint" "Capacitor_SMD:C_0603_1608Metric"
       (at 58.42 71.12 0)
       (hide yes)
@@
         (font
           (size 1.27 1.27))))
-    (property "Footprint" ""
+    (property "Footprint" "Capacitor_SMD:C_0603_1608Metric"
       (at 45.72 71.12 0)
       (hide yes)
@@
         (font
           (size 1.27 1.27))))
-    (property "Footprint" ""
+    (property "Footprint" "Resistor_SMD:R_0603_1608Metric"
       (at 104.14 86.36 0)
       (hide yes)
@@
         (font
           (size 1.27 1.27))))
-    (property "Footprint" ""
+    (property "Footprint" "Resistor_SMD:R_0603_1608Metric"
       (at 104.14 91.44 0)
       (hide yes)
@@
         (font
           (size 1.27 1.27))))
-    (property "Footprint" ""
+    (property "Footprint" "odrive_footprints:L_CommonMode_Murata_DLW32SH101XF2"
       (at 104.14 104.14 0)
       (hide yes)
@@
         (font
           (size 1.27 1.27))))
-    (property "Footprint" ""
+    (property "Footprint" "Resistor_SMD:R_0603_1608Metric"
       (at 127 106.68 0)
       (hide yes)
@@
         (font
           (size 1.27 1.27))))
-    (property "Footprint" ""
+    (property "Footprint" "Resistor_SMD:R_0603_1608Metric"
       (at 127 119.38 0)
       (hide yes)
@@
         (font
           (size 1.27 1.27))))
-    (property "Footprint" ""
+    (property "Footprint" "Capacitor_SMD:C_0603_1608Metric"
       (at 137.16 114.3 0)
       (hide yes)
@@
         (font
           (size 1.27 1.27))))
-    (property "Footprint" ""
+    (property "Footprint" "Button_Switch_THT:SW_DIP_SPSTx01_Slide_9.78x4.72mm_W7.62mm_P2.54mm"
       (at 127 134.62 0)
       (hide yes)
@@
         (font
           (size 1.27 1.27))))
-    (property "Footprint" ""
+    (property "Footprint" "Package_TO_SOT_SMD:SOT-23"
       (at 167.64 109.22 0)
       (hide yes)
@@
         (font
           (size 1.27 1.27))))
-    (property "Footprint" ""
+    (property "Footprint" "Connector_JST:JST_GH_BM04B-GHS-TBT_1x04-1MP_P1.25mm_Vertical"
       (at 198.12 78.74 0)
       (hide yes)
@@
         (font
           (size 1.27 1.27))))
-    (property "Footprint" ""
+    (property "Footprint" "Connector_JST:JST_GH_BM04B-GHS-TBT_1x04-1MP_P1.25mm_Vertical"
       (at 198.12 99.06 0)
       (hide yes)
@@
         (font
           (size 1.27 1.27))))
-    (property "Footprint" ""
+    (property "Footprint" "Package_TO_SOT_SMD:SOT-23-6"
       (at 99.06 40.64 0)
       (hide yes)
@@
         (font
           (size 1.27 1.27))))
-    (property "Footprint" ""
+    (property "Footprint" "Capacitor_SMD:C_0603_1608Metric"
       (at 81.28 43.18 0)
       (hide yes)
@@
         (font
           (size 1.27 1.27))))
-    (property "Footprint" ""
+    (property "Footprint" "Resistor_SMD:R_0603_1608Metric"
       (at 119.38 53.34 0)
       (hide yes)
@@
         (font
           (size 1.27 1.27))))
-    (property "Footprint" ""
+    (property "Footprint" "Capacitor_SMD:C_0805_2012Metric"
       (at 134.62 43.18 0)
       (hide yes)
@@
           (reference "#PWR017")
           (unit 1)))))
-)
+  (text "5V AUX POWER SWITCH"
+    (at 76.2 27.94 0)
+    (effects (font (size 1.5 1.5)))
+  )
+  (text "CAN TRANSCEIVER"
+    (at 40.64 58.42 0)
+    (effects (font (size 1.5 1.5)))
+  )
+  (text "SPLIT TERMINATION"
+    (at 146.05 132.08 0)
+    (effects (font (size 1.5 1.5)))
+  )
+  (text "CAN CONNECTORS"
+    (at 190.5 67.31 0)
+    (effects (font (size 1.5 1.5)))
+  ))
