File: projects/odrive/kicad/odrive-v4/encoders-gpio.kicad_sch (KiCad schematic)
At the start: 55 parts, among them J10 ENC_M1_JST-GH, J11 ENC_SPI_JST-GH, J12 GPIO_2x4, J9 ENC_M0_JST-GH, U30 TPS2553DBV, U31 TPS2553DBV, U35 SN74LVC2G17, U36 SN74LVC2G17, U37 SN74LVC2G17, U38 TPD4E05U06, U39 TPD4E05U06, U40 SN74LVC1G125, U41 TPD4E05U06, U42 TPD1E10B06

Commit message: Make the v4 schematic sheets readable, netlist-invariant
The verified v4 schematic was electrically perfect and visually unreadable:
connectivity lived in labels stuck on pins, text overlapped, and parts sat
on the title block. Reworked all ten block sheets through Konnect: real
wires for local connections, labels kept for power rails and inter-sheet
nets, parts grouped by function, junction dots where wires join.

The invariant was enforced, not assumed: the exported netlist is diffed
against a reference frozen before the rework - 378 components and 283 nets,
identical membership pin by pin - and ERC holds at 0 errors. The lesson
that forced the rework is now a standing gate: numeric oracles (ERC,
netlist diff, overlap counts) all passed on the unreadable version, so
every sheet is also rendered to PNG and looked at before being declared
done.

An interrupted fix round left one known cosmetic issue, documented in
docs/LOG.md: the encoders-gpio GPIO group's reference/value text fields
float ~134mm right of their symbols, over the title block. konnect 0.2.2
has no tool that repositions property fields, so it waits for 0.11.0.
Also adds the fab footprints the sheets reference (MEGA fuse, Phoenix
terminal blocks, CMC) and restores the board file to the blank template -
the aborted layout skeleton was not worth keeping.
Parts:
- C140, C141, C142, C143, C144, C145, C148, C149, C150, C151, C152, C153, C154, C155, C156, C157, C158: footprint (none) -> Capacitor_SMD:C_0603_1608Metric
- C146, C147: footprint (none) -> Capacitor_SMD:C_0805_2012Metric
- J10, J11, J9: footprint (none) -> Connector_JST:JST_GH_BM06B-GHS-TBT_1x06-1MP_P1.25mm_Vertical
- J12: footprint (none) -> Connector_PinHeader_2.54mm:PinHeader_2x04_P2.54mm_Vertical
- R180, R181, R182, R183, R184, R185, R186, R187, R188, R189, R190, R191, R192, R193, R194, R195, R196, R197, R198, R199, R200, R201: footprint (none) -> Resistor_SMD:R_0603_1608Metric
- U30, U31, U35, U36, U37: footprint (none) -> Package_TO_SOT_SMD:SOT-23-6
- U38, U39, U41: footprint (none) -> Package_SON:USON-10_2.5x1.0mm_P0.5mm
- U40: footprint (none) -> Package_TO_SOT_SMD:SOT-23-5
- U42: footprint (none) -> Diode_SMD:D_SOD-523
Connections:
- no-connect marks 14 -> 12
Other:
- moved on the sheet: C148, C149, C150, C151, C152, J12, R197, R198, R199, R200, R201, U41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
