File: projects/odrive/kicad/odrive-v4/rails.kicad_sch (KiCad schematic)
At the start: 43 parts, among them J5 FAN 12V 150mA MAX, U20 LM5164DDA, U21 LMR51430, U22 TLV75533PDBV, U23 TPS7A2033DBV, U25 74LVC1G06, U26 TLV7031DBV, U27 74LVC1G08, U28 TPS3840DL30

Commit message: Make the v4 schematic sheets readable, netlist-invariant
The verified v4 schematic was electrically perfect and visually unreadable:
connectivity lived in labels stuck on pins, text overlapped, and parts sat
on the title block. Reworked all ten block sheets through Konnect: real
wires for local connections, labels kept for power rails and inter-sheet
nets, parts grouped by function, junction dots where wires join.

The invariant was enforced, not assumed: the exported netlist is diffed
against a reference frozen before the rework - 378 components and 283 nets,
identical membership pin by pin - and ERC holds at 0 errors. The lesson
that forced the rework is now a standing gate: numeric oracles (ERC,
netlist diff, overlap counts) all passed on the unreadable version, so
every sheet is also rendered to PNG and looked at before being declared
done.

An interrupted fix round left one known cosmetic issue, documented in
docs/LOG.md: the encoders-gpio GPIO group's reference/value text fields
float ~134mm right of their symbols, over the title block. konnect 0.2.2
has no tool that repositions property fields, so it waits for 0.11.0.
Also adds the fab footprints the sheets reference (MEGA fuse, Phoenix
terminal blocks, CMC) and restores the board file to the blank template -
the aborted layout skeleton was not worth keeping.
Other:
- moved on the sheet: C110, C111, C112, C113, C114, C115, C116, C117, C118, C119, C120, C122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
