File: projects/odrive/kicad/odrive-v4/motorcell-m0.kicad_sch (KiCad schematic)
At the start: 57 parts, among them J2 M0 A/B/C, Q10 NVMFS5C628NL, Q11 NVMFS5C628NL, Q12 NVMFS5C628NL, Q13 NVMFS5C628NL, Q14 NVMFS5C628NL, Q15 NVMFS5C628NL, Q16 NVMFS5C628NL, Q17 NVMFS5C628NL, Q18 NVMFS5C628NL, Q19 NVMFS5C628NL, Q20 NVMFS5C628NL, Q21 NVMFS5C628NL, U3 DRV8353RS

Commit message: Import the v4 netlist onto a 4-layer board, checkpoint before placement
update_pcb_from_schematic (konnect 0.11.0, live IPC, single undo commit)
lands all 378 footprints with 283 nets and zero conflicts. Getting there
took three tries worth of fixes, all kept: the project fp-lib-table now
registers the 18 standard footprint libraries the sheets reference (the
kicad wrapper's KICAD10_FOOTPRINT_DIR is invisible to project resolution,
same story as the symbol libraries); the seven current shunts move to the
real R_Shunt_Vishay_WSK2512_6332Metric_T2.66mm kelvin footprint (the
T1_T2 name the builder invented does not exist); the OV-latch 74LVC1G74
moves to TSSOP-8 (no DCU footprint in this library snapshot - order the
DCT variant); and the SO3 solder jumpers drop the RoundedPad variant
whose custom-shape pads KiCad 10's typed IPC placement path refuses.
Board outline 120x80mm rounded, In1/In2.Cu added file-based after
learning that adding them with pcbnew open gets clobbered by its next
save. Placement not started - components sit stacked at the import
default.
Parts:
- R22, R23, R24: footprint Resistor_SMD:R_Shunt_Vishay_WSK2512_6332Metric_T1_T2 -> Resistor_SMD:R_Shunt_Vishay_WSK2512_6332Metric_T2.66mm
Changed lines of the file:
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@@
       )
     )
-    (property "Footprint" "Resistor_SMD:R_Shunt_Vishay_WSK2512_6332Metric_T1_T2"
+    (property "Footprint" "Resistor_SMD:R_Shunt_Vishay_WSK2512_6332Metric_T2.66mm"
       (at 140.97 88.9 0)
       (hide yes)
@@
       )
     )
-    (property "Footprint" "Resistor_SMD:R_Shunt_Vishay_WSK2512_6332Metric_T1_T2"
+    (property "Footprint" "Resistor_SMD:R_Shunt_Vishay_WSK2512_6332Metric_T2.66mm"
       (at 209.55 88.9 0)
       (hide yes)
@@
       )
     )
-    (property "Footprint" "Resistor_SMD:R_Shunt_Vishay_WSK2512_6332Metric_T1_T2"
+    (property "Footprint" "Resistor_SMD:R_Shunt_Vishay_WSK2512_6332Metric_T2.66mm"
       (at 278.13 88.9 0)
       (hide yes)
