File: projects/odrive/kicad/odrive-v4/motorcell-m1.kicad_sch (KiCad schematic)
At the start: 57 parts, among them J3 M1 A/B/C, Q30 NVMFS5C628NL, Q31 NVMFS5C628NL, Q32 NVMFS5C628NL, Q33 NVMFS5C628NL, Q34 NVMFS5C628NL, Q35 NVMFS5C628NL, Q36 NVMFS5C628NL, Q37 NVMFS5C628NL, Q38 NVMFS5C628NL, Q39 NVMFS5C628NL, Q40 NVMFS5C628NL, Q41 NVMFS5C628NL, U4 DRV8353RS

Commit message: Import the v4 netlist onto a 4-layer board, checkpoint before placement
update_pcb_from_schematic (konnect 0.11.0, live IPC, single undo commit)
lands all 378 footprints with 283 nets and zero conflicts. Getting there
took three tries worth of fixes, all kept: the project fp-lib-table now
registers the 18 standard footprint libraries the sheets reference (the
kicad wrapper's KICAD10_FOOTPRINT_DIR is invisible to project resolution,
same story as the symbol libraries); the seven current shunts move to the
real R_Shunt_Vishay_WSK2512_6332Metric_T2.66mm kelvin footprint (the
T1_T2 name the builder invented does not exist); the OV-latch 74LVC1G74
moves to TSSOP-8 (no DCU footprint in this library snapshot - order the
DCT variant); and the SO3 solder jumpers drop the RoundedPad variant
whose custom-shape pads KiCad 10's typed IPC placement path refuses.
Board outline 120x80mm rounded, In1/In2.Cu added file-based after
learning that adding them with pcbnew open gets clobbered by its next
save. Placement not started - components sit stacked at the import
default.
Parts:
- R52, R53, R54: footprint Resistor_SMD:R_Shunt_Vishay_WSK2512_6332Metric_T1_T2 -> Resistor_SMD:R_Shunt_Vishay_WSK2512_6332Metric_T2.66mm
Changed lines of the file:
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@@
       )
     )
-    (property "Footprint" "Resistor_SMD:R_Shunt_Vishay_WSK2512_6332Metric_T1_T2"
+    (property "Footprint" "Resistor_SMD:R_Shunt_Vishay_WSK2512_6332Metric_T2.66mm"
       (at 127 88.9 0)
       (hide yes)
@@
       )
     )
-    (property "Footprint" "Resistor_SMD:R_Shunt_Vishay_WSK2512_6332Metric_T1_T2"
+    (property "Footprint" "Resistor_SMD:R_Shunt_Vishay_WSK2512_6332Metric_T2.66mm"
       (at 195.58 88.9 0)
       (hide yes)
@@
       )
     )
-    (property "Footprint" "Resistor_SMD:R_Shunt_Vishay_WSK2512_6332Metric_T1_T2"
+    (property "Footprint" "Resistor_SMD:R_Shunt_Vishay_WSK2512_6332Metric_T2.66mm"
       (at 264.16 88.9 0)
       (hide yes)
