File: projects/odrive/kicad/odrive-v4-mono/odrive-v4-mono.kicad_sch (KiCad schematic)
At the start: 4 parts

Commit message: Add odrive-v4-mono: single-axis variant for faster iteration
Copies the v4 project and removes the MotorCell M1 sheet instance, so the
board drives one motor (the sim-racing wheel case, where the second axis was
dead weight: ~12 FETs, a DRV8353, shunts and a phase terminal of unused BOM).
The dual-axis odrive-v4 stays untouched as the robotics variant.

Verified at every step against the oracles rather than assumed:
- netlist: 325 components, exactly the 57 M1 refs fewer than dual (382)
- ERC: 0 errors; the only new warnings vs the dual baseline are 16
  isolated_pin_label for the now-unpaired M1_* globals (spare MCU pins)
- board synced live via update_pcb_from_schematic (which preserves
  schematic-orphaned footprints as board-only, so the 57 M1 footprints were
  then deleted explicitly and the count re-checked: 325 = netlist)
- placement: verdict pass, zero courtyard overlaps

H1-H4 mounting holes now carry the M3 footprint in both variants - the
board-loop workflow had added the symbols with an empty Footprint field,
which broke netlist preflight ('KiCad netlist node is missing footprint').
Their board positions came from schematic coordinates (off-board at x=8),
found by grid search over free courtyard space; the metric that works is
Chebyshev distance, since courtyard overlap is a bbox test on both axes -
euclidean 'clearance' kept placing holes diagonally into corners of
neighbouring courtyards.

The unreferenced motorcell-m1.kicad_sch copy is dropped from the new dir.
Known state: left half of the 170x115 outline is now empty; shrinking the
outline needs the full-width logic band re-placed first. Zones inherited and
refilled; routing still pending.
Other:
- removed sheet MotorCell M1
Changed lines of the file:
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@@
     )
   )
-  (sheet
-    (at 127 124.46)
-    (size 50.8 78.74)
-    (fields_autoplaced)
-    (stroke
-      (width 0.1524)
-      (type solid)
-    )
-    (fill
-      (color 0 0 0 0.0)
-    )
-    (property "Sheetname" "MotorCell M1"
-      (at 127 123.66 0)
-    )
-    (property "Sheetfile" "motorcell-m1.kicad_sch"
-      (at 127 203.6 0)
-    )
-    (instances
-      (project "odrive-v4"
-        (path "/8f2a1c40-5d3b-4a6e-9c17-0b5e2d84f731"
-          (page "4")
-        )
-      )
-    )
-  )
-  (sheet
+    (sheet
     (at 38.1 88.9)
     (size 63.5 96.52)
