File: projects/odrive/kicad/odrive-v4-mono/can.kicad_sch (KiCad schematic)
At the start: 17 parts, among them J7 JST-GH-4 CAN, J8 JST-GH-4 CAN, SW1 CAN_TERM, U32 TPS2553DBV, U34 TCAN1042HGV

Commit message: Checkpoint ODrive 56 V recovery and modular handoff
Preserve corrected schematics, local libraries, partial PCB routing, firmware diagnostics, analysis tools and the independent modular-study handoff. The board remains incomplete with 381 unconnected items and 415 DRC warnings.

Validation: 52 host tests, ARM component compilation, schematic/PCB parity, native copper preservation, DRC, STEP export, Python lint, shellcheck and nix fmt. Known Konnect-generated schematic whitespace is retained. No fabrication or hardware validation is claimed.
Parts:
- U32: symbol /home/aldo/Dev/aldoborrero/cad/.claude/worktrees/odrive/projects/odrive/kicad/odrive-v4/odrive-v4-symbols:TPS2553DBV -> odrive-mono:TPS2553DBV; MPN (none) -> TPS2553DBVR; Manufacturer (none) -> Texas Instruments
Connections:
- net +5V: now also U32.1 (IN); no longer U32.6 (IN)
- net AUX_5V: now also U32.6 (OUT); no longer U32.1 (OUT)
- net at U32.4 (~{FAULT}): no longer R129.1
- net at U32.5 (ILIM): now also R129.1
Changed lines of the file:
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@@
           (unit 1)))))
   (symbol
-    (lib_id "/home/aldo/Dev/aldoborrero/cad/.claude/worktrees/odrive/projects/odrive/kicad/odrive-v4/odrive-v4-symbols:TPS2553DBV")
+    (lib_id "odrive-mono:TPS2553DBV")
     (at 99.06 40.64 0)
     (unit 1)
@@
         (font
           (size 1.27 1.27))))
-    (property "Datasheet" ""
+    (property "Datasheet" "https://www.ti.com/lit/ds/symlink/tps2553.pdf"
       (at 99.06 40.64 0)
       (hide yes)
@@
         (path "/ad37970d-e2d0-40ab-96f7-27502fcb978c"
           (reference "U32")
-          (unit 1)))))
+          (unit 1))))
+    (property "MPN" "TPS2553DBVR"
+    	(at 99.06 40.64 0)
+    	(hide yes)
+    	(effects
+    		(font
+    			(size 1.27 1.27)
+    		)
+    	)
+    )
+    (property "Manufacturer" "Texas Instruments"
+    	(at 99.06 40.64 0)
+    	(hide yes)
+    	(effects
+    		(font
+    			(size 1.27 1.27)
+    		)
+    	)
+    ))
   (symbol
     (lib_id "Device:C")
