File: projects/odrive/kicad/odrive-v4-mono/motorcell-m0.kicad_sch (KiCad schematic)
At the start: 57 parts, among them J2 M0 A/B/C, Q10 NVMFS5C628NL, Q11 NVMFS5C628NL, Q12 NVMFS5C628NL, Q13 NVMFS5C628NL, Q14 NVMFS5C628NL, Q15 NVMFS5C628NL, Q16 NVMFS5C628NL, Q17 NVMFS5C628NL, Q18 NVMFS5C628NL, Q19 NVMFS5C628NL, Q20 NVMFS5C628NL, Q21 NVMFS5C628NL, U3 DRV8353RS

Commit message: Checkpoint ODrive 56 V recovery and modular handoff
Preserve corrected schematics, local libraries, partial PCB routing, firmware diagnostics, analysis tools and the independent modular-study handoff. The board remains incomplete with 381 unconnected items and 415 DRC warnings.

Validation: 52 host tests, ARM component compilation, schematic/PCB parity, native copper preservation, DRC, STEP export, Python lint, shellcheck and nix fmt. Known Konnect-generated schematic whitespace is retained. No fabrication or hardware validation is claimed.
Parts:
- added C200: 1uF 25V X7R, Capacitor_SMD:C_0603_1608Metric, symbol Device:C
- added C201: 470nF 25V X7R, Capacitor_SMD:C_0603_1608Metric, symbol Device:C
- added C202: 2.2uF 100V X7R, Capacitor_SMD:C_1210_3225Metric, symbol Device:C
- added C203: 100nF 100V X7R, Capacitor_SMD:C_0603_1608Metric, symbol Device:C
- added C204: 10nF 50V X7R, Capacitor_SMD:C_0603_1608Metric, symbol Device:C
- added C205: 3.3nF 100V C0G, Capacitor_SMD:C_0603_1608Metric, symbol Device:C
- added C206: 100nF 50V X7R, Capacitor_SMD:C_0603_1608Metric, symbol Device:C
- added C207: 22uF 50V X7R, Capacitor_SMD:C_1210_3225Metric, symbol Device:C
- added D200: STPS1H100A, Diode_SMD:D_SMA, symbol Device:D_Schottky
- added L200: 330uH, Inductor_SMD:L_Bourns_SRR1260, symbol Device:L
- added R202: 4.7k, Resistor_SMD:R_0603_1608Metric, symbol Device:R
- added R203: 470k, Resistor_SMD:R_0805_2012Metric, symbol Device:R
- added R204: 470k, Resistor_SMD:R_0603_1608Metric, symbol Device:R
- added R205: 5.62k, Resistor_SMD:R_0603_1608Metric, symbol Device:R
- added R206: 1k, Resistor_SMD:R_0603_1608Metric, symbol Device:R
- added R207: 130k, Resistor_SMD:R_0805_2012Metric, symbol Device:R
- C30, C31: value 1uF -> 1uF 25V X7R
- C32: value 1uF 100V X7R -> 22uF 50V X7R; Design_note (none) -> VM local bypass: require at least 10uF effective at 18V, in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
- C33: value 100nF -> 100nF 50V X7R
- Q10, Q11, Q12, Q13, Q14, Q15, Q16, Q17, Q18, Q19, Q20, Q21: value NVMFS5C628NL -> BSC027N10NS5; footprint Package_SO:PowerPAK_SO-8_Single -> odrive-mono:Infineon_PG-TSON-8-3; symbol Transistor_FET:Q_NMOS_GDS -> Transistor_FET:Q_NMOS_SSSGD_AvalancheRated; Design_note (none) -> 100V selection; verify losses, SOA, cooling and mask apertu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; MPN (none) -> BSC027N10NS5ATMA1; MPN_56V (none) -> BSC027N10NS5ATMA1; Manufacturer (none) -> Infineon
- U3: symbol /home/aldo/Dev/aldoborrero/cad/.claude/worktrees/odrive/projects/odrive/kicad/odrive-v4/odrive-v4-symbols:DRV8353RS -> odrive-mono:DRV8353RSRGZ; Design_note (none) -> Integrated buck supplies M0_VM only, nominal 16.55 V before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; MPN (none) -> DRV8353RSRGZR; Manufacturer (none) -> Texas Instruments
Connections:
- net DCBUS: now also Q10.5 (D), Q11.5 (D), Q14.5 (D), Q15.5 (D), Q18.5 (D), Q19.5 (D), U3.43 (VIN), U3.6 (VDRAIN), C202.1, C203.1, R203.1; no longer C32.1, C33.1, Q10.2 (D), Q11.2 (D), Q14.2 (D), Q15.2 (D), Q18.2 (D), Q19.2 (D), U3.4 (VM), U3.5 (VDRAIN)
- net DRV_ENABLE: now also U3.33 (ENABLE); no longer U3.27 (ENABLE)
- net GND: now also U3.1 (GND), U3.27 (AGND), U3.41 (DGND), C200.2, C201.2, C202.2, C203.2, C207.2, D200.2 (A), R204.2, R206.2; no longer U3.22 (GND), U3.39 (VIN), U3.40 (nSHDN)
- net M0_A: now also Q10.1 (S), Q10.2 (S), Q11.1 (S), Q11.2 (S), Q12.5 (D), Q13.5 (D), U3.9 (SHA); no longer Q12.2 (D), Q13.2 (D), U3.7 (SHA)
- net M0_AH: now also U3.34 (INHA); no longer U3.29 (INHA)
- net M0_AL: now also U3.35 (INLA); no longer U3.30 (INLA)
- net M0_B: now also Q14.1 (S), Q14.2 (S), Q15.1 (S), Q15.2 (S), Q16.5 (D), Q17.5 (D), U3.16 (SHB); no longer Q16.2 (D), Q17.2 (D), U3.12 (SHB)
- net M0_BH: now also U3.36 (INHB); no longer U3.31 (INHB)
- net M0_BL: now also U3.37 (INLB); no longer U3.32 (INLB)
- net M0_C: now also Q18.1 (S), Q18.2 (S), Q19.1 (S), Q19.2 (S), Q20.5 (D), Q21.5 (D), U3.19 (SHC); no longer Q20.2 (D), Q21.2 (D), U3.17 (SHC)
- net M0_CH: now also U3.38 (INHC); no longer U3.33 (INHC)
- net M0_CL: now also U3.39 (INLC); no longer U3.34 (INLC)
- net M0_CPH: now also U3.4 (CPH); no longer U3.2 (CPH)
- net M0_CPL: now also U3.3 (CPL); no longer U3.1 (CPL)
- net M0_GHA: now also U3.8 (GHA); no longer U3.6 (GHA)
- net M0_GHA1: now also Q10.4 (G); no longer Q10.1 (G)
- net M0_GHA2: now also Q11.4 (G); no longer Q11.1 (G)
- net M0_GHB: now also U3.17 (GHB); no longer U3.11 (GHB)
- net M0_GHB1: now also Q14.4 (G); no longer Q14.1 (G)
- net M0_GHB2: now also Q15.4 (G); no longer Q15.1 (G)
- net M0_GHC: now also U3.18 (GHC); no longer U3.16 (GHC)
- net M0_GHC1: now also Q18.4 (G); no longer Q18.1 (G)
- net M0_GHC2: now also Q19.4 (G); no longer Q19.1 (G)
- net M0_GLA: now also U3.10 (GLA); no longer U3.8 (GLA)
- net M0_GLA1: now also Q12.4 (G); no longer Q12.1 (G)
- net M0_GLA2: now also Q13.4 (G); no longer Q13.1 (G)
- net M0_GLB: now also U3.15 (GLB); no longer U3.13 (GLB)
- net M0_GLB1: now also Q16.4 (G); no longer Q16.1 (G)
- net M0_GLB2: now also Q17.4 (G); no longer Q17.1 (G)
- net M0_GLC: now also U3.20 (GLC); no longer U3.18 (GLC)
- net M0_GLC1: now also Q20.4 (G); no longer Q20.1 (G)
- net M0_GLC2: now also Q21.4 (G); no longer Q21.1 (G)
- net M0_SN_A: now also U3.12 (SNA); no longer U3.10 (SNA)
- net M0_SN_B: now also U3.13 (SNB); no longer U3.15 (SNB)
- net M0_SN_C: now also U3.22 (SNC); no longer U3.20 (SNC)
- net M0_SO2: now also U3.23 (SOC); no longer U3.25 (SOC)
- net M0_SO3: now also U3.25 (SOA); no longer U3.23 (SOA)
- net M0_SP_A: now also U3.11 (SPA); no longer U3.9 (SPA)
- net M0_SP_C: now also U3.21 (SPC); no longer U3.19 (SPC)
- net M0_SRC_A: now also Q12.1 (S), Q12.2 (S), Q13.1 (S), Q13.2 (S)
- net M0_SRC_B: now also Q16.1 (S), Q16.2 (S), Q17.1 (S), Q17.2 (S)
- net M0_SRC_C: now also Q20.1 (S), Q20.2 (S), Q21.1 (S), Q21.2 (S)
- net M0_VCP: now also U3.7 (VCP); no longer U3.3 (VCP)
- net M0_VGLS: now also U3.2 (VGLS); no longer U3.21 (VGLS)
- net M0_nCS: now also U3.32 (nSCS); no longer U3.38 (nSCS)
- net SPI3_MISO: now also U3.29 (SDO), R202.2; no longer U3.37 (SDO)
- net SPI3_MOSI: now also U3.30 (SDI); no longer U3.36 (SDI)
- net SPI3_SCK: now also U3.31 (SCLK); no longer U3.35 (SCLK)
- net VCC: now also R202.1
- net M0_BUCK_SW: now reaches U3.42 (SW)
- net M0_BUCK_SW: now also C204.2, D200.1 (K), L200.1, R207.1
- net M0_BUCK_VCC: now reaches U3.44 (VCC)
- net M0_BUCK_VCC: now also C201.1
- net M0_BUCK_BST: now reaches U3.45 (BST)
- net M0_BUCK_BST: now also C204.1
- net M0_BUCK_RCL: now reaches U3.46 (RCL)
- net M0_BUCK_RCL: now also R204.1
- net M0_BUCK_RT: now reaches U3.47 (RT/SD)
- net M0_BUCK_RT: now also R203.2
- net M0_BUCK_FB: now reaches U3.48 (FB)
- net M0_BUCK_FB: now also C206.2, R205.2, R206.1
- new net: C205.1, C206.1, R207.2
- new net M0_DVDD: C200.1, U3.40 (DVDD)
- new net M0_VM: C205.2, C207.1, C32.1, C33.1, L200.2, R205.1, U3.5 (VM)
- no-connect marks 8 -> 0
Other:
- note added: "U3 BUCK: dedicated gate-driver supply, ~16.5 V 12 V logic / brake rail remains separate Ripple injection: LM5008A datasheet Figure 12 See docs/v4-mono-56v-driver-supply.md for limits"
