File: projects/odrive/kicad/odrive-v4-mono/rails.kicad_sch (KiCad schematic)
At the start: 43 parts, among them J5 FAN 12V 150mA MAX, U20 LM5164DDA, U21 LMR51430, U22 TLV75533PDBV, U23 TPS7A2033DBV, U25 74LVC1G06, U26 TLV7031DBV, U27 74LVC1G08, U28 TPS3840DL30

Commit message: Checkpoint ODrive 56 V recovery and modular handoff
Preserve corrected schematics, local libraries, partial PCB routing, firmware diagnostics, analysis tools and the independent modular-study handoff. The board remains incomplete with 381 unconnected items and 415 DRC warnings.

Validation: 52 host tests, ARM component compilation, schematic/PCB parity, native copper preservation, DRC, STEP export, Python lint, shellcheck and nix fmt. Known Konnect-generated schematic whitespace is retained. No fabrication or hardware validation is claimed.
Parts:
- added C214: 10nF 100V C0G, Capacitor_SMD:C_0603_1608Metric, symbol Device:C
- added C215: 330pF 50V C0G, Capacitor_SMD:C_0603_1608Metric, symbol Device:C
- added R215: 68.1k, Resistor_SMD:R_0805_2012Metric, symbol Device:R
- C113: value 100nF 25V -> 2.2nF 50V X7R; Design_note (none) -> LM5164 BST-SW: 1.5-2.5nF permitted; TI SNVSAU4D tables 4-1 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; Tolerance (none) -> 5%
- L1: footprint Inductor_SMD:L_12x12mm_H8mm -> Inductor_SMD:L_Wuerth_WE-PD-Typ-LS; DCR_max_ohm_20C (none) -> 0.110; Design_note (none) -> No vias or sensitive traces below the body. Qualify effecti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; Height_max_mm (none) -> 10; Isat_10pct_typ_A (none) -> 3.1; LCSC (none) -> C6463690; MPN (none) -> 7447709101; Manufacturer (none) -> Wurth Elektronik; Operating_voltage_max_V (none) -> 120; Tolerance (none) -> 20%
- L2: value 4.7uH -> 6.8uH; footprint Inductor_SMD:L_Taiyo-Yuden_NR-50xx -> odrive-mono:Coilcraft_XAL7070_682; Assembly_note (none) -> Marked winding start at pad 1 / SW5; see F.Fab bar.; DCR_max_ohm_25C (none) -> 0.01962; Design_note (none) -> Hot inductance, fault overshoot and losses require qualific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; Height_max_mm (none) -> 7; Isat_30pct_typ_A_25C (none) -> 12.8; LCSC (none) -> C3911753; MPN (none) -> XAL7070-682MEC; Manufacturer (none) -> Coilcraft; Operating_voltage_max_V (none) -> 60; Tolerance (none) -> 20%
- R110, R111: Tolerance (none) -> 1%
- R118: value 301k -> 75k; Design_note (none) -> LM5164 nominal CCM frequency about 367kHz with 12.108V divi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; Tolerance (none) -> 1%
- U20: MPN (none) -> LM5164DDAR; Manufacturer (none) -> Texas Instruments
- U21: value LMR51430 -> LMR51430XFDDCR; footprint Package_TO_SOT_SMD:SOT-23-6 -> odrive-mono:TI_DDC0006A; Control_mode (none) -> FPWM; Design_note (none) -> TI device table specifies 500kHz FPWM. Catalogue descriptio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; LCSC (none) -> C5219260; MPN (none) -> LMR51430XFDDCR; Manufacturer (none) -> Texas Instruments; Switching_frequency_Hz (none) -> 500000
- U25: value 74LVC1G06 -> 74LVC1G07; symbol 74xGxx:74LVC1G06 -> 74xGxx:74LVC1G07; Design_note (none) -> Open-drain non-inverting: rail PG low asserts nFAULT; high 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; MPN (none) -> SN74LVC1G07DBVR; Manufacturer (none) -> Texas Instruments
- U27: MPN (none) -> SN74LVC1G08DBVR; Manufacturer (none) -> Texas Instruments
- U28: symbol /home/aldo/Dev/aldoborrero/cad/.claude/worktrees/odrive/projects/odrive/kicad/odrive-v4/odrive-v4-symbols:TPS3840DL30 -> odrive-mono:TPS3840DL30DBV; MPN (none) -> TPS3840DL30DBVR; Manufacturer (none) -> Texas Instruments
Connections:
- net +12V: now also C214.2
- net FB12: now also C215.2
- net GND: now also U28.3 (GND); no longer U28.2 (GND)
- net SW12: now also R215.1
- net VCC: now also U28.2 (VDD); no longer U28.5 (VDD)
- net PG_ALL renamed RAILS_OK
- new net RIPPLE12: C214.1, C215.1, R215.2
