File: projects/odrive/kicad/odrive-v4-mono/sensing.kicad_sch (KiCad schematic)
At the start: 67 parts, among them U10 TLV9062, U11 TMUX1204, U12 TLV7031, U13 TLV431, U14 74LVC1G04, U15 74LVC1G08

Commit message: Checkpoint ODrive 56 V recovery and modular handoff
Preserve corrected schematics, local libraries, partial PCB routing, firmware diagnostics, analysis tools and the independent modular-study handoff. The board remains incomplete with 381 unconnected items and 415 DRC warnings.

Validation: 52 host tests, ARM component compilation, schematic/PCB parity, native copper preservation, DRC, STEP export, Python lint, shellcheck and nix fmt. Known Konnect-generated schematic whitespace is retained. No fabrication or hardware validation is claimed.
Parts:
- removed R96: 4.7k, Resistor_SMD:R_0603_1608Metric, symbol Device:R
- removed U13: TLV431, Package_TO_SOT_SMD:SOT-23, symbol /home/aldo/Dev/aldoborrero/cad/.claude/worktrees/odrive/projects/odrive/kicad/o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
- added C208, C209, C213: 100nF 16V X7R, Capacitor_SMD:C_0603_1608Metric, symbol Device:C
- added C210: 1uF 16V X7R, Capacitor_SMD:C_0603_1608Metric, symbol Device:C
- added C211: 100pF 50V C0G, Capacitor_SMD:C_0603_1608Metric, symbol Device:C
- added R208: 47k, Resistor_SMD:R_0603_1608Metric, symbol Device:R
- added R209, R214: 1k, Resistor_SMD:R_0603_1608Metric, symbol Device:R
- added R210, R213: 10k, Resistor_SMD:R_0603_1608Metric, symbol Device:R
- added R211: 10.5k, Resistor_SMD:R_1206_3216Metric, symbol Device:R
- added unit 2 of U12
- added U13: REF35125QDBVR, Package_TO_SOT_SMD:SOT-23-6, symbol Reference_Voltage:REF35125QDBVR
- added U56: 74LVC1G74, Package_SO:VSSOP-8_2.3x2mm_P0.5mm, symbol odrive-mono:74LVC1G74DCU
- added U57: 74LVC1G11, Package_TO_SOT_SMD:SOT-23-6, symbol odrive-mono:74LVC1G11DBV
- added U59: 74LVC1G08, Package_TO_SOT_SMD:SOT-23-5, symbol 74xGxx:74LVC1G08
- C62: value 100nF -> 1uF 16V X7R; Design_note (none) -> Keep total cathode capacitance below 1 nF including parasit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; Effective capacitance (none) -> 0.1 uF minimum, 10 uF maximum; ESR <= 0.4 ohm; Tolerance (none) -> 10%
- R70: value 10k | 18k -> 10.5k; footprint Resistor_SMD:R_0603_1608Metric -> Resistor_SMD:R_1206_3216Metric; Design_note (none) -> One of two series 10.5k divider resistors; ratio 22:1. Veri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; Power (none) -> 0.25 W minimum at 70 C; TCR (none) -> 25 ppm/K max; Tolerance (none) -> 0.1%; Voltage (none) -> 200 V minimum working
- R71: Design_note (none) -> 56 V mono OV correction; exact MPN and full temperature qua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; TCR (none) -> 25 ppm/K max; Tolerance (none) -> 0.1%
- R93: value 12k | 15.4k -> 455k; footprint Resistor_SMD:R_0603_1608Metric -> Resistor_SMD:R_1206_3216Metric; Design_note (none) -> 56 V mono OV correction; exact MPN and full temperature qua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; Power (none) -> 0.25 W minimum at 70 C; TCR (none) -> 25 ppm/K maximum; Tolerance (none) -> 0.1%; Working voltage (none) -> 200 V minimum
- R94: Design_note (none) -> 56 V mono OV correction; exact MPN and full temperature qua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; TCR (none) -> 25 ppm/K maximum; Tolerance (none) -> 0.1%
- R95: value 130k -> 301k; Design_note (none) -> 56 V mono OV correction; exact MPN and full temperature qua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; TCR (none) -> 25 ppm/K maximum; Tolerance (none) -> 0.1%
- U11: symbol /home/aldo/Dev/aldoborrero/cad/.claude/worktrees/odrive/projects/odrive/kicad/odrive-v4/odrive-v4-symbols:TMUX1204 -> odrive-mono:TMUX1204DGS; MPN (none) -> TMUX1204DGSR; Manufacturer (none) -> Texas Instruments
- U12: value TLV7031 -> TLV3201AIDBVR; symbol Comparator:TLV7031DBV -> odrive-mono:TLV3201AIDBVR; Design_note (none) -> Nominal OV ~60 V / ~55 V; full threshold/delay qualificatio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; MPN (none) -> TLV3201AIDBVR; Manufacturer (none) -> Texas Instruments
- U14: MPN (none) -> SN74LVC1G04DBVR; Manufacturer (none) -> Texas Instruments
- U15: MPN (none) -> SN74LVC1G08DBVR; Manufacturer (none) -> Texas Instruments
Connections:
- net ADC_AUX: now also U11.8 (D); no longer U11.7 (D)
- net AGND: now also U11.3 (GND); no longer C62.2, R94.2, U11.5 (GND)
- net AVCC: now also U11.5 (EN); no longer U11.10 (VDD)
- net BRAKE_ISENSE: now also U11.4 (S3); no longer U11.9 (S3)
- net DCBUS: now also R93.1, R211.1; no longer R70.1
- net DRV_ENABLE: now also R209.1, R210.1
- net DRV_EN_MCU: now also R208.1, U56.1 (C)
- net GND: now also C62.2, R94.2, C208.2, C209.2, C210.2, C211.2, C213.2, R208.2, R209.2, R214.2, U12.2 (GND), U13.1 (GND), U13.2 (GND), U56.4 (GND), U57.2 (GND), U59.3 (GND); no longer U12.2 (V-)
- net GPIO_6: now also U11.10 (A1); no longer U11.3 (A1)
- net M0_MOTOR_THERM_F: now also U11.2 (S1); no longer U11.1 (S1)
- net M1_MOTOR_THERM_F: now also U11.9 (S2); no longer U11.2 (S2)
- net MUX_A0: now also U11.1 (A0); no longer U11.4 (A0)
- net OV_LATCH_N: now also U57.6 (C); no longer U15.2
- net OV_SENSE: now also C211.1
- net USB_VBUS_SENSE: now also U11.7 (S4); no longer U11.8 (S4)
- net VBUS_S_BUF: no longer R93.1
- net VCC: now also C208.1, C209.1, C210.1, C213.1, U12.5 (VCC), U13.3 (EN), U13.4 (VIN), U56.2 (D), U56.7 (~{PRE}), U56.8 (VCC), U57.5 (VCC), U59.5 (VCC); no longer U12.5 (V+)
- net VREF_OV: now also U13.6 (VREF)
- new net BRK_OK: R213.1, R214.1, U59.2
- new net BRK_OK_FB: R213.2
- new net DRV_ARMED: U15.2, U56.5 (Q)
- new net DRV_ARM_CLEAR_N: U56.6 (~{CLR}), U57.4 (Y)
- new net DRV_ENABLE_FB: R210.2
- new net DRV_RUN_READY: U57.1 (A), U59.4
- new net NRST: U57.3 (B)
- new net RAILS_OK: U59.1
- new net VBUS_DIV_TOP: R211.2, R70.1
- no-connect marks 1 -> 3
Other:
- note added: "BRAKE PERMISSION / MOTOR INHIBIT BRK_OK LOW clears the motor arm latch through U59/U57. Recovery requires a fresh DRV_EN_MCU rising edge. PC7 reads BRK_OK_FB through R213; configure input/no-pull. Permission does not prove resistor continuity or energy capacity."
- note added: "MONO 56 V INDEPENDENT OV INPUT R93 senses DCBUS directly; R94 returns to GND. U13 = REF35125QDBVR, 1.25 V, powered from VCC. U12 = TLV3201AIDBVR; C211 filters OV_SENSE. Ideal external-network trip/release: 60.01 / 55.03 V. ADC divider remains 22:1; firmware port required. Tolerance, startup, transient and brake qualification remain open."
- note added: "MONO ENABLE INTERLOCK OV / rail-good loss / brake permission loss / reset clears U56. Recovery requires a NEW rising PB12 request. U15 also disables immediately when PB12 is low. PC6 reads DRV_ENABLE; PC7 reads BRK_OK; firmware port required."
- moved on the sheet: C61, C62
